File: led_driver.sch (KiCad schematic (older format))
At the start: 307 parts, among them IC1 DM13A, IC10 DM13A, IC11 DM13A, IC12 DM13A, IC14 74LS138, IC2 DM13A, IC3 DM13A, IC4 DM13A, IC5 DM13A, IC6 DM13A, IC7 DM13A, IC8 DM13A, IC9 DM13A, P1 CONN_10, P2 5V, T1 MOSFET_P, T2 MOSFET_P, T3 MOSFET_P, T4 MOSFET_P, T5 MOSFET_P, T6 MOSFET_P, T7 MOSFET_P, T8 MOSFET_P

Commit message: finished manual routing
Parts:
- B0, B1, B10, B11, B12, B13, B14, B15, B16, B17, B18, B19, B2, B20, B21, B22, B23, B24, B25, B26, B27, B28, B29, B3, B30, B31, B32, B33, B34, B35, B36, B37, B38, B39, B4, B40, B41, B42, B43, B44, B45, B46, B47, B48, B49, B5, B50, B51, B52, B53, B54, B55, B56, B57, B58, B59, B6, B60, B61, B62, B63, B7, B8, B9, G0, G1, G10, G11, G12, G13, G14, G15, G16, G17, G18, G19, G2, G20, G21, G22, G23, G24, G25, G26, G27, G28, G29, G3, G30, G31, G32, G33, G34, G35, G36, G37, G38, G39, G4, G40, G41, G42, G43, G44, G45, G46, G47, G48, G49, G5, G50, G51, G52, G53, G54, G55, G56, G57, G58, G59, G6, G60, G61, G62, G63, G7, G8, G9, L1_ROW1, L1_ROW2, L1_ROW3, L1_ROW4, L1_ROW5, L1_ROW6, L1_ROW7, L1_ROW8, L2_ROW1, L2_ROW2, L2_ROW3, L2_ROW4, L2_ROW5, L2_ROW6, L2_ROW7, L2_ROW8, L3_ROW1, L3_ROW2, L3_ROW3, L3_ROW4, L3_ROW5, L3_ROW6, L3_ROW7, L3_ROW8, L4_ROW1, L4_ROW2, L4_ROW3, L4_ROW4, L4_ROW5, L4_ROW6, L4_ROW7, L4_ROW8, L5_ROW1, L5_ROW2, L5_ROW3, L5_ROW4, L5_ROW5, L5_ROW6, L5_ROW7, L5_ROW8, L6_ROW1, L6_ROW2, L6_ROW3, L6_ROW4, L6_ROW5, L6_ROW6, L6_ROW7, L6_ROW8, L7_ROW1, L7_ROW2, L7_ROW3, L7_ROW4, L7_ROW5, L7_ROW6, L7_ROW7, L7_ROW8, L8_ROW1, L8_ROW2, L8_ROW3, L8_ROW4, L8_ROW5, L8_ROW6, L8_ROW7, L8_ROW8, R0, R1, R10, R11, R12, R13, R14, R15, R16, R17, R18, R19, R2, R20, R21, R22, R23, R24, R25, R26, R27, R28, R29, R3, R30, R31, R32, R33, R34, R35, R36, R37, R38, R39, R4, R40, R41, R42, R43, R44, R45, R46, R47, R48, R49, R5, R50, R51, R52, R53, R54, R55, R56, R57, R58, R59, R6, R60, R61, R62, R63, R7, R8, R9: footprint (none) -> Connectors:Pin_d1.0mm_L10.0mm_LooseFit
- C1, C2, C3, C4, C5, C6, C7, C8: footprint (none) -> Capacitors_THT:CP_Radial_D8.0mm_P5.00mm
- IC1, IC10, IC11, IC12, IC2, IC3, IC4, IC5, IC6, IC7, IC8, IC9: footprint (none) -> Housings_DIP:DIP-24_W7.62mm_Socket_LongPads
- IC14: footprint (none) -> Housings_DIP:DIP-16_W7.62mm_Socket_LongPads
- P1: footprint (none) -> Pin_Headers:Pin_Header_Straight_1x10_Pitch2.54mm
- P2: footprint (none) -> Connectors_WAGO:WAGO_734_2pin_Straight_RuggedPads
- R_1, R_10, R_11, R_12, R_13, R_2, R_3, R_4, R_5, R_6, R_7, R_8, R_9: footprint (none) -> Resistors_THT:R_Axial_DIN0309_L9.0mm_D3.2mm_P12.70mm_Horizontal
- R_14, R_15, R_16, R_17, R_18, R_19, R_20: footprint ~ -> Resistors_THT:R_Axial_DIN0309_L9.0mm_D3.2mm_P12.70mm_Horizontal
- T1, T2, T3, T4, T5, T6, T7, T8: footprint ~ -> TO_SOT_Packages_THT:TO-220-3_Horizontal
