File: led_driver.kicad_pcb (KiCad board)
At the start: 2 copper layers, 296 x 296 mm, 312 parts, among them IC1 DM13A, IC10 DM13A, IC11 DM13A, IC12 DM13A, IC14 74LS138, IC2 DM13A, IC3 DM13A, IC4 DM13A, IC5 DM13A, IC6 DM13A, IC7 DM13A, IC8 DM13A, IC9 DM13A, P1 CONN_10, P2 5V, T1 MOSFET_P, T2 MOSFET_P, T3 MOSFET_P, T4 MOSFET_P, T5 MOSFET_P, T6 MOSFET_P, T7 MOSFET_P, T8 MOSFET_P

Commit message: finished manual routing
Parts:
- removed ? (x5): , Connectors:1pin
- moved R_2 13.0 mm to (92.8, 40.0), turned to 180 degrees
- moved C5 0.50 mm to (176.8, 61.5)
Routing:
- net GND: track 0.00 -> 571.6 mm
- net VCC: track 0.00 -> 512.2 mm
- net Net-(L4_ROW1-Pad1): track 0.00 -> 315.9 mm
- net Net-(L3_ROW1-Pad1): track 0.00 -> 315.7 mm
- net Net-(L8_ROW1-Pad1): track 0.00 -> 314.7 mm
- net Net-(L2_ROW1-Pad1): track 0.00 -> 314.4 mm
- net Net-(L5_ROW1-Pad1): track 0.00 -> 313.8 mm
- net Net-(L6_ROW1-Pad1): track 0.00 -> 313.7 mm
- net Net-(L7_ROW1-Pad1): track 0.00 -> 313.5 mm
- net Net-(L1_ROW1-Pad1): track 284.0 -> 317.8 mm

Commit message: finished pcb
Routing:
- net GND: track 571.6 -> 1915.3 mm, vias 0 -> 3
- net CLOCK: track 0.00 -> 1005.3 mm, vias 0 -> 7
- net EN: track 0.00 -> 960.0 mm, vias 0 -> 9
- net LAT: track 0.00 -> 913.1 mm, vias 0 -> 6
- net VCC: track 512.2 -> 1324.6 mm, vias 0 -> 2
- net Net-(B40-Pad1): track 0.00 -> 441.3 mm, vias 0 -> 3
- net Net-(B0-Pad1): track 0.00 -> 393.3 mm, vias 0 -> 3
- net Net-(B8-Pad1): track 0.00 -> 375.5 mm, vias 0 -> 1
- net Net-(G15-Pad1): track 0.00 -> 372.2 mm, vias 0 -> 2
- net GREEN: track 0.00 -> 368.5 mm, vias 0 -> 2
- net Net-(G7-Pad1): track 0.00 -> 342.6 mm, vias 0 -> 3
- net Net-(B16-Pad1): track 0.00 -> 272.8 mm, vias 0 -> 5
- net Net-(B56-Pad1): track 0.00 -> 272.1 mm
- net Net-(B24-Pad1): track 0.00 -> 272.0 mm, vias 0 -> 5
- net Net-(G55-Pad1): track 0.00 -> 272.0 mm, vias 0 -> 1
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- added copper zone on B.Cu, net GND
- added copper zone on F.Cu, net VCC
Other:
- board text added: "8x8x8 3D LED Driver Board, 23 nov. 2017, Edwin Mol"
